Commit message: Added code for different kinds of joints

File: my_robot.urdf (robot description, URDF)
Before this commit: robot my_robot, 2 links, 1 joints
Links:
- added link third_link; visual box length=0.2 radius=0.1 0.1 0.1
Joints:
- added joint second_third_joint: type fixed, parent second_link, child third_link, origin xyz=0 0 0 rpy=0 0 0
- joint base_second_joint: axis (none) -> 0 0 1; limit (none) -> lower=-1.57 upper=1.57 effort=100 velocity=100; type fixed -> revolute
