Commit message: progres

File: section_3/s3_activity.urdf (robot description, URDF)
Before this commit: robot my_robot, 0 links, 0 joints
Links:
- added link base_link; visual box size=0.6 0.4 0.2
- added link left_link; visual cylinder length=0.2 radius=0.1
Joints:
- added joint base_left_joint: type revolute, parent base_link, child left_link, origin xyz=0 0 0.2 rpy=0 0 0, axis 0 0 1, limit lower=-1.57 upper=1.57 effort=100 velocity=100

Commit message: progress

File: section_3/s3_activity.urdf (robot description, URDF)
Before this commit: robot my_robot, 2 links, 1 joints
Links:
- added link center_link; visual sphere radius=0.075
- added link right_link; visual cylinder length=0.075 radius=0.15
- link left_link: geometry visual cylinder length=0.075 radius=0.15
Joints:
- added joint base_center_joint: type fixed, parent base_link, child center_link, origin xyz=0.25 0 -0.075 rpy=0 0 0
- added joint base_right_joint: type revolute, parent base_link, child left_link, origin xyz=-0.2 -0.25 0 rpy=1.57 0 0, axis 0 0 1, limit lower=-1.57 upper=1.57 effort=100 velocity=100
- joint base_left_joint: child left_link -> right_link; origin xyz=0 0 0.2 rpy=0 0 0 -> xyz=-0.2 0.25 0 rpy=1.57 0 0
